File: tests/fixtures/design_lint/pcb-keepout-rule-area.kicad_pcb (KiCad board)
At the start: 2 copper layers, 0 parts

Commit message: Add source-mapped RF antenna keepout lint
Parts:
- added U1: Probe_Module, RF_Module:Probe_Module, F.Cu at (20.0, 20.0)
- added U2: Probe_Module, RF_Module:Probe_Module, B.Cu at (30.0, 25.0)
- added U3: Probe_Module, RF_Module:Probe_Module, F.Cu at (40.0, 40.0)
Changed lines of the file:
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@@
   (setup (pad_to_mask_clearance 0))
   (net 0 "")
+  (net 1 "RF_FEED")
+  (footprint "RF_Module:Probe_Module"
+    (layer "F.Cu")
+    (at 20 20 90)
+    (property "Reference" "U1"
+      (at 20 18 90)
+      (layer "F.SilkS")
+      (effects (font (size 1 1) (thickness 0.15)))
+    )
+    (property "Value" "Probe_Module"
+      (at 20 22 90)
+      (layer "F.Fab")
+      (effects (font (size 1 1) (thickness 0.15)))
+    )
+    (attr smd)
+    (pad "1" smd rect
+      (at 1 0)
+      (size 1 1)
+      (layers "F.Cu" "F.Mask" "F.Paste")
+      (net 1 "RF_FEED")
+    )
+  )
+  (footprint "RF_Module:Probe_Module"
+    (layer "B.Cu")
+    (at 30 25 270)
+    (property "Reference" "U2"
+      (at 30 27 270)
+      (layer "B.SilkS")
+      (effects (font (size 1 1) (thickness 0.15)) (justify mirror))
+    )
+    (property "Value" "Probe_Module"
+      (at 30 23 270)
+      (layer "B.Fab")
+      (effects (font (size 1 1) (thickness 0.15)) (justify mirror))
+    )
+    (attr smd)
+    (pad "1" smd rect
+      (at -1 0)
+      (size 1 1)
+      (layers "B.Cu" "B.Mask" "B.Paste")
+      (net 1 "RF_FEED")
+    )
+  )
+  (footprint "RF_Module:Probe_Module"
+    (layer "F.Cu")
+    (at 40 40 30)
+    (property "Reference" "U3"
+      (at 40 38 30)
+      (layer "F.SilkS")
+      (effects (font (size 1 1) (thickness 0.15)))
+    )
+    (property "Value" "Probe_Module"
+      (at 40 42 30)
+      (layer "F.Fab")
+      (effects (font (size 1 1) (thickness 0.15)))
+    )
+    (attr smd)
+    (pad "1" smd rect
+      (at 1 0)
+      (size 1 1)
+      (layers "F.Cu" "F.Mask" "F.Paste")
+      (net 1 "RF_FEED")
+    )
+  )
   (zone
     (net 0)
@@
       )
     )
+  )
+  (zone
+    (net 0)
+    (net_name "")
+    (layers "F.Cu" "B.Cu")
+    (name "SYNTHETIC_ANTENNA_KEEPOUT_BACK")
+    (hatch edge 0.5)
+    (keepout
+      (tracks not_allowed)
+      (vias not_allowed)
+      (pads not_allowed)
+      (copperpour not_allowed)
+      (footprints allowed)
+    )
+    (polygon
+      (pts
+        (xy 30 25)
+        (xy 30 28)
+        (xy 32 28)
+        (xy 32 25)
+      )
+    )
+  )
+  (zone
+    (net 0)
+    (net_name "")
+    (layers "F.Cu" "B.Cu")
+    (name "SYNTHETIC_ANTENNA_KEEPOUT_ANGLED")
+    (hatch edge 0.5)
+    (keepout
+      (tracks not_allowed)
+      (vias not_allowed)
+      (pads not_allowed)
+      (copperpour not_allowed)
+      (footprints allowed)
+    )
+    (polygon
+      (pts
+        (xy 40 40)
+        (xy 42.598076 38.5)
+        (xy 43.098076 39.366025)
+        (xy 40.5 40.866025)
+      )
+    )
