File: tests/fixtures/design_lint/component-peer-power-assignment-native/fault.kicad_sch (KiCad schematic)
At the start: 2 parts, among them U1 Synthetic power module, U2 Synthetic power module

Commit message: Add comparable peer pin lint gates
Connections:
- net DATA renamed SYNTHETIC_NET_A
- net SYNTHETIC_NET_A: no longer U2.1 (IO)
- net VOUT_A renamed SYNTHETIC_NET_C
- net VOUT_B renamed SYNTHETIC_NET_D
- new net SYNTHETIC_NET_B: U2.1 (VDD)
Other:
- title: Synthetic power-output peer control -> Synthetic power-pin assignment peer fault
Changed lines of the file:
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@@
 (kicad_sch (version 20231120) (generator "eeschema")
   (paper "A4")
-  (title_block (title "Synthetic power-output peer control")
+  (title_block (title "Synthetic power-pin assignment peer fault")
     (comment 1 "NOT FOR MANUFACTURE - tooling fixture"))
   (symbol (lib_id "Synthetic:PowerModule") (at 88.9 78.74 0) (unit 1)
@@
     (pin "1")
     (pin "2")
-    (instances (project "Synthetic peer power-output fixture" (path "/58fe9fab-a929-4a44-a7fd-b83188082220" (reference "U1") (unit 1))))
+    (instances (project "Synthetic peer power-pin assignment fixture" (path "/58fe9fab-a929-4a44-a7fd-b83188082219" (reference "U1") (unit 1))))
   )
   (symbol (lib_id "Synthetic:PowerModuleAlias") (at 165.1 78.74 0) (unit 1)
@@
     (pin "1")
     (pin "2")
-    (instances (project "Synthetic peer power-output fixture" (path "/58fe9fab-a929-4a44-a7fd-b83188082220" (reference "U2") (unit 1))))
+    (instances (project "Synthetic peer power-pin assignment fixture" (path "/58fe9fab-a929-4a44-a7fd-b83188082219" (reference "U2") (unit 1))))
   )
   (wire (pts (xy 83.82 78.74) (xy 73.66 78.74))
     (stroke (width 0) (type default))
 )
-  (label "DATA" (at 73.66 78.74 0)
+  (label "SYNTHETIC_NET_A" (at 73.66 78.74 0)
     (effects (font (size 1.27 1.27)) (justify left bottom))
 )
@@
     (stroke (width 0) (type default))
 )
-  (label "DATA" (at 149.86 78.74 0)
+  (label "SYNTHETIC_NET_B" (at 149.86 78.74 0)
     (effects (font (size 1.27 1.27)) (justify left bottom))
 )
@@
     (stroke (width 0) (type default))
 )
-  (label "VOUT_A" (at 104.14 78.74 0)
+  (label "SYNTHETIC_NET_C" (at 104.14 78.74 0)
     (effects (font (size 1.27 1.27)) (justify left bottom))
 )
@@
     (stroke (width 0) (type default))
 )
-  (label "VOUT_B" (at 180.34 78.74 0)
+  (label "SYNTHETIC_NET_D" (at 180.34 78.74 0)
     (effects (font (size 1.27 1.27)) (justify left bottom))
 )
