File: tests/fixtures/design_lint/four-port-db9-returns/control.kicad_sch (KiCad schematic)
At the start: 4 parts, among them J1 Synthetic DB9 connector, J2 Synthetic DB9 connector, J3 Synthetic DB9 connector, J4 Synthetic DB9 connector

Commit message: Add comparable peer pin lint gates
Connections:
- net 0V PWM renamed COMMON_RETURN
Changed lines of the file:
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@@
     (stroke (width 0) (type default))
 )
-  (label "0V PWM" (at 43.18 96.52 0)
+  (label "COMMON_RETURN" (at 43.18 96.52 0)
     (effects (font (size 1.27 1.27)) (justify left bottom))
 )
@@
     (stroke (width 0) (type default))
 )
-  (label "0V PWM" (at 43.18 91.44 0)
+  (label "COMMON_RETURN" (at 43.18 91.44 0)
     (effects (font (size 1.27 1.27)) (justify left bottom))
 )
@@
     (stroke (width 0) (type default))
 )
-  (label "0V PWM" (at 99.06 96.52 0)
+  (label "COMMON_RETURN" (at 99.06 96.52 0)
     (effects (font (size 1.27 1.27)) (justify left bottom))
 )
@@
     (stroke (width 0) (type default))
 )
-  (label "0V PWM" (at 99.06 91.44 0)
+  (label "COMMON_RETURN" (at 99.06 91.44 0)
     (effects (font (size 1.27 1.27)) (justify left bottom))
 )
@@
     (stroke (width 0) (type default))
 )
-  (label "0V PWM" (at 154.94 96.52 0)
+  (label "COMMON_RETURN" (at 154.94 96.52 0)
     (effects (font (size 1.27 1.27)) (justify left bottom))
 )
@@
     (stroke (width 0) (type default))
 )
-  (label "0V PWM" (at 154.94 91.44 0)
+  (label "COMMON_RETURN" (at 154.94 91.44 0)
     (effects (font (size 1.27 1.27)) (justify left bottom))
 )
@@
     (stroke (width 0) (type default))
 )
-  (label "0V PWM" (at 210.82 96.52 0)
+  (label "COMMON_RETURN" (at 210.82 96.52 0)
     (effects (font (size 1.27 1.27)) (justify left bottom))
 )
@@
     (stroke (width 0) (type default))
 )
-  (label "0V PWM" (at 210.82 91.44 0)
+  (label "COMMON_RETURN" (at 210.82 91.44 0)
     (effects (font (size 1.27 1.27)) (justify left bottom))
 )
