File: tests/fixtures/design_lint/four-port-db9-returns/fault.kicad_sch (KiCad schematic)
At the start: 4 parts, among them J1 Synthetic DB9 connector, J2 Synthetic DB9 connector, J3 Synthetic DB9 connector, J4 Synthetic DB9 connector

Commit message: Add comparable peer pin lint gates
Connections:
- net 0V PWM 1 renamed RETURN_PORT_1
- net 0V PWM 2 renamed RETURN_PORT_2
- net 0V PWM 3 renamed RETURN_PORT_3
- net 0V PWM 4 renamed RETURN_PORT_4
Changed lines of the file:
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@@
     (stroke (width 0) (type default))
 )
-  (label "0V PWM 1" (at 43.18 96.52 0)
+  (label "RETURN_PORT_1" (at 43.18 96.52 0)
     (effects (font (size 1.27 1.27)) (justify left bottom))
 )
@@
     (stroke (width 0) (type default))
 )
-  (label "0V PWM 1" (at 43.18 91.44 0)
+  (label "RETURN_PORT_1" (at 43.18 91.44 0)
     (effects (font (size 1.27 1.27)) (justify left bottom))
 )
@@
     (stroke (width 0) (type default))
 )
-  (label "0V PWM 2" (at 99.06 96.52 0)
+  (label "RETURN_PORT_2" (at 99.06 96.52 0)
     (effects (font (size 1.27 1.27)) (justify left bottom))
 )
@@
     (stroke (width 0) (type default))
 )
-  (label "0V PWM 2" (at 99.06 91.44 0)
+  (label "RETURN_PORT_2" (at 99.06 91.44 0)
     (effects (font (size 1.27 1.27)) (justify left bottom))
 )
@@
     (stroke (width 0) (type default))
 )
-  (label "0V PWM 3" (at 154.94 96.52 0)
+  (label "RETURN_PORT_3" (at 154.94 96.52 0)
     (effects (font (size 1.27 1.27)) (justify left bottom))
 )
@@
     (stroke (width 0) (type default))
 )
-  (label "0V PWM 3" (at 154.94 91.44 0)
+  (label "RETURN_PORT_3" (at 154.94 91.44 0)
     (effects (font (size 1.27 1.27)) (justify left bottom))
 )
@@
     (stroke (width 0) (type default))
 )
-  (label "0V PWM 4" (at 210.82 96.52 0)
+  (label "RETURN_PORT_4" (at 210.82 96.52 0)
     (effects (font (size 1.27 1.27)) (justify left bottom))
 )
@@
     (stroke (width 0) (type default))
 )
-  (label "0V PWM 4" (at 210.82 91.44 0)
+  (label "RETURN_PORT_4" (at 210.82 91.44 0)
     (effects (font (size 1.27 1.27)) (justify left bottom))
 )
