File: tests/fixtures/design_lint/component-inventory-footprint-identity/control.kicad_pcb (KiCad board)
At the start: 2 copper layers, 1 part, among them U1 Probe_Module

Commit message: feat(pcb): add schematic-board value consistency lint
Parts:
- U1: value Probe_Module -> Synthetic identity probe
Changed lines of the file:
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@@
       (effects (font (size 1 1) (thickness 0.15)))
     )
-    (property "Value" "Probe_Module"
+    (property "Value" "Synthetic identity probe"
       (at 20 22 0)
       (layer "F.Fab")
