File: tests/fixtures/design_lint/unconnected-named-connector-pins/return-fault.kicad_sch (KiCad schematic)
At the start: 1 part, among them J1 Synthetic named connector

Commit message: fix: use validated KiCad source for connector pin fixtures
Parts:
- removed J1: Synthetic named connector, Synthetic:Connector, symbol Synthetic:NamedConnector
- added J1: Synthetic named connector, Synthetic:Component, symbol Lint:PowerRoleComponent
Connections:
- net +3V3: now also J1.1 (VDD)
Other:
- title: Synthetic unconnected connector return pin -> Synthetic connected connector power pins
Changed lines of the file:
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@@
 (kicad_sch (version 20231120) (generator "eeschema")
   (paper "A4")
-  (title_block (title "Synthetic unconnected connector return pin")
+  (title_block (title "Synthetic connected connector power pins")
     (comment 1 "NOT FOR MANUFACTURE - tooling regression fixture"))
-  (symbol (lib_id "Synthetic:NamedConnector") (at 63.5 101.6 0) (unit 1)
+  (symbol (lib_id "Lint:PowerRoleComponent") (at 63.5 101.6 0) (unit 1)
     (in_bom yes) (on_board yes) (dnp no)
     (property "Reference" "J1" (at 63.5 88.9 0) (effects (font (size 1.27 1.27)) (justify left)))
     (property "Value" "Synthetic named connector" (at 63.5 91.44 0) (effects (font (size 1.27 1.27)) (justify left)))
-    (property "Footprint" "Synthetic:Connector" (at 63.5 101.6 0) (effects (font (size 1.27 1.27)) hide))
+    (property "Footprint" "Synthetic:Component" (at 63.5 101.6 0) (effects (font (size 1.27 1.27)) hide))
     (property "Datasheet" "" (at 63.5 101.6 0) (effects (font (size 1.27 1.27)) hide))
     (pin "1")
     (pin "2")
     (instances (project "synthetic-unconnected-connector-return"
-      (path "/41000001-0000-4000-8000-000000000001" (reference "J1") (unit 1)))))
+      (path "/00000011-0000-4000-8000-000000000001" (reference "J1") (unit 1)))))
   (wire (pts (xy 50.8 104.14) (xy 43.18 104.14))
     (stroke (width 0) (type default))
@@
     (effects (font (size 1.27 1.27)) (justify left bottom))
 )
-  (sheet_instances (page "1"))
+  (sheet_instances (path "/" (page "1")))
 )
